File: dbmbyhd.kicad_pcb (KiCad board)
At the start: 2 copper layers, 16.8 x 13.6 mm, 16 parts, among them J1 Conn_01x02, J2 Conn_01x04, J3 Conn_01x02, J4 Conn_01x03, U1 rt9525gqw

Commit message: rev1
Routing:
- net GND: vias 3 -> 4
Other:
- board text added: "DBMBYHD rev1"
- board text removed: "DBMBYHD rev0"
Changed lines of the file:
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@@
-(kicad_pcb (version 20171130) (host pcbnew 5.1.5+dfsg1-2)
+(kicad_pcb (version 20171130) (host pcbnew 5.1.5+dfsg1-2+b1)
   (general
     (thickness 1.6)
     (drawings 6)
-    (tracks 72)
+    (tracks 73)
     (zones 0)
     (modules 16)
@@
     (effects (font (size 1 1) (thickness 0.15)) (justify mirror))
   )
-  (gr_text "DBMBYHD rev0" (at 148.5265 101.6) (layer B.SilkS)
+  (gr_text "DBMBYHD rev1" (at 148.5265 101.6) (layer B.SilkS)
     (effects (font (size 1 1) (thickness 0.15)) (justify mirror))
   )
@@
   (via (at 149.159347 104.391847) (size 0.8) (drill 0.4) (layers F.Cu B.Cu) (net 1))
   (via (at 148.9075 100.5205) (size 0.8) (drill 0.4) (layers F.Cu B.Cu) (net 1))
+  (via (at 147.1 95.95) (size 0.8) (drill 0.4) (layers F.Cu B.Cu) (net 1))
   (segment (start 145.631 98.5775) (end 145.542 98.5775) (width 0.25) (layer F.Cu) (net 3))
   (segment (start 147.316 100.2625) (end 145.631 98.5775) (width 0.25) (layer F.Cu) (net 3))
